File: electronic/Eagle/quantum/quantun_AnalougeEngine/quantum_AnalougeEngine_V3_0/quantum_AnalougeEngine_V3_0.brd (EAGLE design)
At the start: 171.7 x 107.6 mm, 167 parts, among them IC1 OP275, IC10 NE5532D, IC2 NE5532D, IC3 NE5532D, IC4 OP275, IC5 NE5532D, IC6 NE5532D, IC7 NE5532D, IC8 OP275, IC9 TL072, K5 RELAY_EE2-5NU, K6 RELAY_EE2-5NU, K7 RELAY_EE2-5NU, K8 RELAY_EE2-5NU, U1 NUCLEO-F429ZI, U12 ULN2003, U4 THAT1240, U6 THAT1240, U7 THAT1240, U8 THAT1240

Commit message: - UART6 Transmit implemented - DMA ADC now fully working - implemented OSCmessageINTSend();
Connections:
- net USART6_RX renamed USART6_TX
- net USRAT6_TX renamed USRAT6_RX
Changed lines of the file:
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@@
 <drawing>
 <settings>
-<setting alwaysvectorfont="yes"/>
+<setting alwaysvectorfont="no"/>
 <setting verticaltext="up"/>
 </settings>
@@
 <wire x1="9.9" y1="6.1" x2="12.3" y2="3.7" width="0.3048" layer="1"/>
 </signal>
-<signal name="USART6_RX">
+<signal name="USART6_TX">
 <contactref element="U1" pad="CN12_4"/>
 </signal>
-<signal name="USRAT6_TX">
+<signal name="USRAT6_RX">
 <contactref element="U1" pad="CN12_19"/>
 </signal>
