File: electronic/Eagle/quantum/quantum_PSU/Orbiter_PowerSupply_V1.sch (EAGLE design)
At the start: 18 parts, among them U4 7815, U5 7915

Commit message: Routed quantum_PSU
Parts:
- D1, D2: value 4148_SOD323 -> 4148THT; device C_Sager_Bibliothek:4148_SOD323 -> C_Sager_Bibliothek:4148THT
Connections:
- new net N$6: U$2.2, U$2.4
Changed lines of the file:
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@@
 <part name="C24" library="C_Sager_Bibliothek" library_urn="urn:adsk.eagle:library:560098" deviceset="KONDENSATOR_THT" device="2.5MM" package3d_urn="urn:adsk.eagle:package:1899462/2" value="10nF"/>
 <part name="C25" library="C_Sager_Bibliothek" library_urn="urn:adsk.eagle:library:560098" deviceset="KONDENSATOR_THT" device="2.5MM" package3d_urn="urn:adsk.eagle:package:1899462/2" value="10nF"/>
-<part name="D1" library="C_Sager_Bibliothek" library_urn="urn:adsk.eagle:library:560098" deviceset="4148_SOD323" device="" package3d_urn="urn:adsk.eagle:package:578210/4"/>
-<part name="D2" library="C_Sager_Bibliothek" library_urn="urn:adsk.eagle:library:560098" deviceset="4148_SOD323" device="" package3d_urn="urn:adsk.eagle:package:578210/4"/>
+<part name="D1" library="C_Sager_Bibliothek" library_urn="urn:adsk.eagle:library:560098" deviceset="4148" device="THT" package3d_urn="urn:adsk.eagle:package:2094195/4" value="4148THT"/>
+<part name="D2" library="C_Sager_Bibliothek" library_urn="urn:adsk.eagle:library:560098" deviceset="4148" device="THT" package3d_urn="urn:adsk.eagle:package:2094195/4"/>
 <part name="U$2" library="C_Sager_Bibliothek" library_urn="urn:adsk.eagle:library:560098" deviceset="PRINTTRAFO_30-600-LPI" device="" package3d_urn="urn:adsk.eagle:package:15708166/1"/>
 </parts>
@@
 </segment>
 </net>
+<net name="N$6" class="0">
+<segment>
+<pinref part="U$2" gate="G$1" pin="4"/>
+<wire x1="35.56" y1="137.16" x2="33.02" y2="137.16" width="0.1524" layer="91"/>
+<pinref part="U$2" gate="G$1" pin="2"/>
+<wire x1="33.02" y1="137.16" x2="33.02" y2="127" width="0.1524" layer="91"/>
+<wire x1="33.02" y1="127" x2="35.56" y2="127" width="0.1524" layer="91"/>
+</segment>
+</net>
