File: electronic/Eagle/quantum/quantun_AnalougeEngine/quantum_AnalougeEngine_V4_0/quantum_AnalougeEngine_V4_0.brd (EAGLE design)
At the start: 171.7 x 107.6 mm, 198 parts, among them IC1 OP275, IC2 DAC084S085CIMM_NOPB, IC3 DAC084S085CIMM_NOPB, IC4 OP275, IC5 OP275, IC7 TL072, IC8 OP275, IC9 TL072, K1 K1, K2 K2, K3 K3, K4 K4, K5 RELAY_EE2-5NU, K6 RELAY_EE2-5NU, K7 RELAY_EE2-5NU, K8 RELAY_EE2-5NU, U1 NUCLEO-F429ZI, U12 ULN2003, U4 THAT1240, U6 THAT1240, U7 THAT1240, U8 THAT1240

Commit message: minor updates on quantum_AnlougeEngine_V4_0
Parts:
- removed +15VOK, -15VOK: SMD_LED_0603, C_Sager_Bibliothek:WL-SMCW_0603
- added LED10, LED9: LED_GREEN_SMD, C_Sager_Bibliothek:WL-SMCW_0603
- added TP04: TPTHT, C_Sager_Bibliothek:THT_PIN
- C69: value (none) -> 0.33 uF
- C70: value (none) -> 100 nF
- K5: value RELAY_EE2-5NU -> K5
- K6: value RELAY_EE2-5NU -> K6
- K7: value RELAY_EE2-5NU -> K7
- K8: value RELAY_EE2-5NU -> K8
- LED1, LED2, LED3, LED4, LED5, LED6, LED7, LED8: value SMD_LED_0603 -> LED_BLUE_SMD
- R10, R11, R12, R33, R34, R7, R8, R9: value 500R -> 470R
- STAGE(LEFT), STAGE(RIGHT), VCA1(LEFT), VCA2(RIGHT): value THAT2181S -> THAT2181SO8-US
- moved TP06 16.8 mm to (8.40, 2.80)
- moved R29 14.5 mm to (9.20, 10.8)
- moved R14 14.5 mm to (4.50, 10.8)
- moved TP23 11.5 mm to (14.2, 11.9)
- moved TP09 10.6 mm to (19.2, 11.9)
- moved R77 1.30 mm to (52.7, 7.90)
- moved TP03 1.30 mm to (48.9, 5.00)
- moved TP05 1.30 mm to (54.0, 5.00)
- moved TP18 1.30 mm to (51.4, 5.00)
- moved CONN3 1.17 mm to (19.2, 4.10)
- moved C23 0.40 mm to (62.4, 21.7)
- moved C24 0.40 mm to (62.4, 10.8)
- moved C19 0.30 mm to (59.7, 26.3)
- renumbered L1 to LED1, L2 to LED2, L3 to LED3, L4 to LED4, L5 to LED5, L6 to LED6, L7 to LED7, L8 to LED8, U$1 to U2, U$2 to C69, U$3 to C70, U$4 to U3
Connections:
- new net BOTTOM: TP06.P$1
- net AGND: now also LED9.1, TP04.P$1; no longer +15VOK.1, TP06.P$1
- net N$50: now also LED10.2; no longer -15VOK.2
- net N$52: now also LED9.2; no longer +15VOK.2
- net V-: now also LED10.1; no longer -15VOK.1
Routing:
- net AGND: track 215.1 -> 236.7 mm
- net N$52: track 3.62 -> 23.8 mm
- net V-: track 70.2 -> 78.2 mm
- net S1: track 42.0 -> 37.1 mm
- net CS: track 89.8 -> 92.2 mm
- net +12V: track 484.0 -> 481.5 mm
- net V+: track 155.8 -> 153.8 mm
- net DB4: track 76.3 -> 74.3 mm
- net DAC_OUT2: track 117.9 -> 119.8 mm
- net DAC_OUT1: track 179.8 -> 181.2 mm
- net M1: track 31.3 -> 32.7 mm
- net CS_DAC1: track 123.0 -> 124.3 mm
- net N$58: track 8.86 -> 10.2 mm
- net N$57: track 12.7 -> 13.8 mm
- net DB1: track 110.7 -> 109.7 mm
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- added copper zone on layer 16, net BOTTOM
Other:
- board text added: "AnalougeEngine V4_0"
- board text added: "bottom"
- board text added: "quantum"

Commit message: Clock changed to 8 MHz Crystal. Progress AnalougeEngine (routing 50 %).
Connections:
- new net SWCLK: U1.CN11_15
- new net SWDIO: U1.CN11_13
Changed lines of the file:
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@@
 <drawing>
 <settings>
-<setting alwaysvectorfont="yes"/>
+<setting alwaysvectorfont="no"/>
 <setting verticaltext="up"/>
 </settings>
@@
 </polygon>
 </signal>
+<signal name="SWCLK">
+<contactref element="U1" pad="CN11_15"/>
+</signal>
+<signal name="SWDIO">
+<contactref element="U1" pad="CN11_13"/>
+</signal>
 </signals>
