File: electronic/Eagle/quantum/quantun_AnalougeEngine/quantum_AnalougeEngine_V5_0/quantum_AnalougeEngine_V5_0.sch (EAGLE design)
At the start: 278 parts, among them IC1 OP275, IC10 STM32F767ZIT6, IC11 AD7606BSTZ, IC12 ESDA6V1BC6, IC13 USBLC6-4SC6, IC14 TL072, IC15 TL072, IC16 OP275, IC2 DAC084S085CIMM_NOPB, IC3 DAC084S085CIMM_NOPB, IC4 OP275, IC5 OP275, IC6 LAN8742A-CZ-TR, IC7 TL072, IC8 OP275, IC9 TL072, J1 GWLEX-SMT-S988G_Y, K1 K1, K2 K2, K3 K3, K4 K4, K5 K5, K6 K6, K7 K7, K8 K8, T1 H1102NL, U12 ULN2003, U4 THAT1240, U6 THAT1240, U7 THAT1240, U8 THAT1240, Y1 NX3215SA-32.768K-STD-MUA-8, Y2 NX3225GD-8MHZ-STD-CRA-3, Y3 ABLS2-25.000MHZ-D4YF-T

Commit message: Analouge Engine V5_0 updates...
Parts:
- removed C103: 100nF, C_Sager_Bibliothek:CAPACITOR"
- added C104: 100 nF, passive components:CAPACITOR_0603
- C1, C11, C12, C13, C14, C19, C2, C20, C21, C22, C23, C24, C25, C26, C27, C28, C29, C3, C30, C35, C36, C4, C43, C44, C45, C46, C47, C48, C49, C5, C50, C53, C54, C57, C58, C6, C60, C61, C62, C63, C68, C7, C8, C95, C96, C97, C98: value 100nF -> 100 nF; device C_Sager_Bibliothek:CAPACITOR" -> passive components:CAPACITOR_0603
- C10, C15, C16, C17, C18, C9: device C_Sager_Bibliothek:CAPACITOR" -> passive components:CAPACITOR_0603
- C37, C38, C55, C56: value 22pF -> 22 pF; device C_Sager_Bibliothek:CAPACITOR" -> passive components:CAPACITOR_0603
Connections:
- net +5V: now also C14.1, C36.1; no longer C19.1, C43.1
- net 1V_DAC: now also C22.1; no longer C23.1
- net 1V_DAC_UNBUFFERD: now also C19.1; no longer C20.1
- net AGND: now also C104.2; no longer C103.2
- net L/M_OUT(OUT_STAGE_LEFT): now also C38.2; no longer C37.2
- net N$48: now also C38.1; no longer C37.1
- net N$53: now also C37.1; no longer C38.1
- net N$54: now also C43.1; no longer C45.1
- net N$73: now also C47.1; no longer C48.1
- net N$77: now also C58.1; no longer C60.1
- net N$80: now also C61.1; no longer C63.1
- net R/S_OUT(OUT_STAGE_RIGHT): now also C37.2; no longer C38.2
- net V+: now also C104.1, C12.1, C21.1, C25.1, C27.1, C29.1, C4.1, C45.1, C48.1, C50.1, C54.1, C6.1, C60.1, C63.1, C8.1; no longer C1.1, C11.1, C13.1, C22.1, C26.1, C28.1, C35.1, C47.1, C49.1, C5.1, C53.1, C58.1, C61.1, C68.1, C7.1
- net V-: now also C1.1, C11.1, C13.1, C20.1, C23.1, C26.1, C28.1, C35.1, C49.1, C5.1, C53.1, C68.1, C7.1; no longer C103.1, C12.1, C14.1, C21.1, C25.1, C27.1, C29.1, C36.1, C4.1, C50.1, C54.1, C6.1, C8.1

Commit message: finished Layout AnalougeEngine5_0
Parts:
- IN_LEFT, IN_RIGHT: value 1240 -> THAT1240
- K1: value K1 -> Relay
- K2: value K2 -> Relay
- K3: value K3 -> Relay
- K4: value K4 -> Relay
- K5: value K5 -> Relay; SPICEPREFIX (none) -> B
- K6: value K6 -> Relay; SPICEPREFIX (none) -> B
- K7: value K7 -> Relay
- K8: value K8 -> Relay
- LD1: value LED_BLUE_SMD -> LED_YELOW_SMD; device C_Sager_Bibliothek:LED_BLUE_SMD -> passive components:LED_YELOW_SMD
- LD2: value LED_BLUE_SMD -> LED_RED_SMD; device C_Sager_Bibliothek:LED_BLUE_SMD -> passive components:LED_RED_SMD
- LD3: value LED_BLUE_SMD -> LED_GREEN_SMD; device C_Sager_Bibliothek:LED_BLUE_SMD -> passive components:LED_GREEN_SMD
- LED1, LED2, LED3, LED4, LED5, LED6, LED7, LED8: device C_Sager_Bibliothek:LED_BLUE_SMD -> passive components:LED_BLUE_SMD
- OUT_LEFT, OUT_RIGHT: value 1646 -> THAT1646
- R1, R14, R35, R4, R42, R46, R54, R55, R56, R57, R58, R60, R61, R62, R65, R67, R70, R71, R72, R74, R75, R87: value 10k -> 10 k; device C_Sager_Bibliothek:RESISTOR -> passive components:RESISTOR_0603
- R10, R11, R13, R33, R34, R5, R6, R8, R9: value 680R -> 680 R; device C_Sager_Bibliothek:RESISTOR -> passive components:RESISTOR_0603
- R100, R101, R18, R19, R20, R21, R22, R23, R24, R25, R26, R27, R28, R29, R30, R31, R32, R36, R37, R40, R43, R47, R50, R51, R63, R66, R7, R76, R77, R78, R79, R80, R81, R82, R83, R84, R85, R88, R89, R90, R91, R92, R93, R94, R95, R97, R98, R99: device C_Sager_Bibliothek:RESISTOR -> passive components:RESISTOR_0603
- R12: value 680R -> 680 R; device C_Sager_Bibliothek:RESISTOR -> passive components:RESISTOR_0603; SPICEPREFIX (none) -> R
- R15, R16, R17, R69: value 0R -> 0 R; device C_Sager_Bibliothek:RESISTOR -> passive components:RESISTOR_0603
- R2, R3, R39, R45, R86: value 100k -> 100 k; device C_Sager_Bibliothek:RESISTOR -> passive components:RESISTOR_0603
- R38, R41, R44, R64: value 27k -> 27 k; device C_Sager_Bibliothek:RESISTOR -> passive components:RESISTOR_0603
- R48, R49, R52, R53, R68: value 20k -> 20 k; device C_Sager_Bibliothek:RESISTOR -> passive components:RESISTOR_0603
- R59: value 56k -> 56 k; device C_Sager_Bibliothek:RESISTOR -> passive components:RESISTOR_0603
- R73: value 10k -> 56 k; device C_Sager_Bibliothek:RESISTOR -> passive components:RESISTOR_0603
- Z1: value BZT52C2V0T-7 -> ZENER_DIODE_BZT; device C_Sager_Bibliothek:BZT52C2V0T-7 -> passive components:ZENER_DIODE_BZT

Commit message: BOM CleanUp
Parts:
- LED5: SPICEPREFIX L -> (none)
- R1, R12, R3, R39, R45, R77, R8, R86: SPICEPREFIX R -> (none)
- R28, R30, R36, R37: value 20k -> 20 k
- R7: value 680R -> 680 R; SPICEPREFIX R -> (none)
- R97, R98: value 650 R -> 680 R
