File: electronic/Eagle/quantum/quantun_AnalougeEngine/quantum_AnalougeEngine_V5_0/quantum_AnalougeEngine_V5_0.sch (EAGLE design)
At the start: 278 parts, among them IC1 OP275, IC10 STM32F767ZIT6, IC11 AD7606BSTZ, IC12 ESDA6V1BC6, IC13 USBLC6-4SC6, IC14 TL072, IC15 TL072, IC16 OP275, IC2 DAC084S085CIMM_NOPB, IC3 DAC084S085CIMM_NOPB, IC4 OP275, IC5 OP275, IC6 LAN8742A-CZ-TR, IC7 TL072, IC8 OP275, IC9 TL072, J1 GWLEX-SMT-S988G_Y, K1 Relay, K2 Relay, K3 Relay, K4 Relay, K5 Relay, K6 Relay, K7 Relay, K8 Relay, T1 H1102NL, U12 ULN2003, U4 THAT1240, U6 THAT1240, U7 THAT1240, U8 THAT1240, Y1 NX3215SA-32.768K-STD-MUA-8, Y2 NX3225GD-8MHZ-STD-CRA-3, Y3 ABLS2-25.000MHZ-D4YF-T

Commit message: finished all PCB designs and created output data.
Parts:
- removed ANALOG_VOLT: 90814-0204, electro_mechanical:90814-0204
- added ANALOG_VOLT_IN, ANALOG_VOLT_OUT, DISPLAY2, INSERT_AFTER_GAIN, INSERT_BEFORE_GAIN: 90814-0204, electro_mechanical:90814-0204
- added TP03, TP04, TP05, TP06, TP07, TP08, TP09, TP10: TPTHT, C_Sager_Bibliothek:TPTHT
- renumbered DISPLAY to DISPLAY1
Connections:
- new net L/M_OUT(OUT_STAGE_LEFT)_BEFORE: C38.2, IC11.V5, IC5A.OUT, INSERT_AFTER_GAIN.3, R28.2
- new net N$96: INSERT_BEFORE_GAIN.2, R37.1
- new net N$97: INSERT_BEFORE_GAIN.4, R36.1
- new net PB12: IC10.PB12, TP05.TP
- new net PD10: IC10.PD10, TP08.TP
- new net PD11: IC10.PD11, TP09.TP
- new net PD12: IC10.PD12, TP10.TP
- new net R/S_OUT(OUT_STAGE_RIGHT)_BEFORE: C37.2, IC11.V6, IC5B.OUT, INSERT_AFTER_GAIN.1, R30.2
- new net USART1_RX: DISPLAY2.2, IC10.PB15
- new net USART1_TX: DISPLAY2.1, IC10.PB6
- net +5V: now also DISPLAY2.3
- net A_GND_TO_STAR: now also ANALOG_VOLT_IN.3, ANALOG_VOLT_IN.4, ANALOG_VOLT_OUT.3, ANALOG_VOLT_OUT.4; no longer ANALOG_VOLT.3, ANALOG_VOLT.4
- net DIN_DAC: now also TP04.TP
- net DISPLAY_GND_TO_STAR: now also DISPLAY2.4
- net L/M_OUT(OUT_STAGE_LEFT): now also INSERT_AFTER_GAIN.4; no longer C38.2, IC11.V5, IC5A.OUT, R28.2
- net L/M_OUT(VCA1_OUT): now also INSERT_BEFORE_GAIN.3; no longer R36.1
- net R/S_OUT(OUT_STAGE_RIGHT): now also INSERT_AFTER_GAIN.2; no longer C37.2, IC11.V6, IC5B.OUT, R30.2
- net R/S_OUT(VCA2_OUT): now also INSERT_BEFORE_GAIN.1; no longer R37.1
- net SCLK_DAC: now also TP03.TP
- net USART3_RX: now also TP06.TP
- net USART3_TX: now also TP07.TP
- net V+: now also ANALOG_VOLT_IN.1, ANALOG_VOLT_OUT.1; no longer ANALOG_VOLT.1
- net V-: now also ANALOG_VOLT_IN.2, ANALOG_VOLT_OUT.2; no longer ANALOG_VOLT.2
Other:
- note added: "display1 adapter"
- note added: "display2 adapter"
- note removed: "display adapter"
- moved on the sheet: +12V_OK, +15V_OK, +3V3_OK, +5V_OK, -15V_OK, DIGITAL_VOLT, R100, R101, R15, R16, R17, R69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
