File: electronic/Eagle/quantum/quantun_AnalougeEngine/quantum_AnalougeEngine_V5_0/quantum_AnalougeEngine_V5_0.brd (EAGLE design)
At the start: 210 x 70 mm, 278 parts, among them IC1 OP275, IC10 STM32F767ZIT6, IC11 AD7606BSTZ, IC12 ESDA6V1BC6, IC13 USBLC6-4SC6, IC14 TL072, IC15 TL072, IC16 OP275, IC2 DAC084S085CIMM_NOPB, IC3 DAC084S085CIMM_NOPB, IC4 OP275, IC5 OP275, IC6 LAN8742A-CZ-TR, IC7 TL072, IC8 OP275, IC9 TL072, J1 GWLEX-SMT-S988G_Y, K1 K1, K2 K2, K3 K3, K4 K4, K5 K5, K6 K6, K7 K7, K8 K8, T1 H1102NL, U12 ULN2003, U4 THAT1240, U6 THAT1240, U7 THAT1240, U8 THAT1240, Y1 NX3215SA-32.768K-STD-MUA-8, Y2 NX3225GD-8MHZ-STD-CRA-3, Y3 ABLS2-25.000MHZ-D4YF-T

Commit message: finished Layout AnalougeEngine5_0
Parts:
- IN_LEFT, IN_RIGHT: value 1240 -> THAT1240
- K1: value K1 -> Relay
- K2: value K2 -> Relay
- K3: value K3 -> Relay
- K4: value K4 -> Relay
- K5: value K5 -> Relay
- K6: value K6 -> Relay
- K7: value K7 -> Relay
- K8: value K8 -> Relay
- LD1: value LED_BLUE_SMD -> LED_YELOW_SMD; device C_Sager_Bibliothek:WL-SMCW_0603 -> passive components:WL-SMCW_0603
- LD2: value LED_BLUE_SMD -> LED_RED_SMD; device C_Sager_Bibliothek:WL-SMCW_0603 -> passive components:WL-SMCW_0603
- LD3: value LED_BLUE_SMD -> LED_GREEN_SMD; device C_Sager_Bibliothek:WL-SMCW_0603 -> passive components:WL-SMCW_0603
- LED1, LED2, LED3, LED4, LED5, LED6, LED7, LED8: device C_Sager_Bibliothek:WL-SMCW_0603 -> passive components:WL-SMCW_0603
- OUT_LEFT, OUT_RIGHT: value 1646 -> THAT1646
- R1, R14, R35, R4, R42, R46, R54, R55, R56, R57, R58, R60, R61, R62, R65, R67, R70, R71, R72, R74, R75, R87: value 10k -> 10 k; device C_Sager_Bibliothek:R0603 -> passive components:R0603
- R10, R11, R12, R13, R33, R34, R5, R6, R8, R9: value 680R -> 680 R; device C_Sager_Bibliothek:R0603 -> passive components:R0603
- R100, R101, R18, R19, R20, R21, R22, R23, R24, R25, R26, R27, R28, R29, R30, R31, R32, R36, R37, R40, R43, R47, R50, R51, R63, R66, R7, R76, R77, R78, R79, R80, R81, R82, R83, R84, R85, R88, R89, R90, R91, R92, R93, R94, R95, R97, R98, R99: device C_Sager_Bibliothek:R0603 -> passive components:R0603
- R15, R16, R17, R69: value 0R -> 0 R; device C_Sager_Bibliothek:R0603 -> passive components:R0603
- R2, R3, R39, R45, R86: value 100k -> 100 k; device C_Sager_Bibliothek:R0603 -> passive components:R0603
- R38, R41, R44, R64: value 27k -> 27 k; device C_Sager_Bibliothek:R0603 -> passive components:R0603
- R48, R49, R52, R53, R68: value 20k -> 20 k; device C_Sager_Bibliothek:R0603 -> passive components:R0603
- R59: value 56k -> 56 k; device C_Sager_Bibliothek:R0603 -> passive components:R0603
- R73: value 10k -> 56 k; device C_Sager_Bibliothek:R0603 -> passive components:R0603
- Z1: value BZT52C2V0T-7 -> ZENER_DIODE_BZT; device C_Sager_Bibliothek:SODFL1608X65N -> passive components:SODFL1608X65N
- moved +15V_OK 59.7 mm to (103.9, 51.7)
- moved -15V_OK 59.7 mm to (111.2, 51.8)
- moved R97 59.7 mm to (114.3, 51.8)
- moved R98 59.7 mm to (107.0, 51.8), turned to 0 degrees
- moved R64 4.00 mm to (49.8, 15.9)
- moved R66 4.00 mm to (46.7, 15.9)
- moved R44 3.90 mm to (49.7, 25.1)
- moved R63 3.90 mm to (46.6, 25.1)
- moved R36 1.08 mm to (49.4, 27.8)
- moved C30 0.70 mm to (49.2, 14.0)
- moved C37 0.70 mm to (50.6, 11.6)
- moved IC5 0.70 mm to (44.0, 11.7)
- moved R28 0.70 mm to (39.2, 12.6)
- moved R30 0.70 mm to (48.7, 11.6)
- moved R37 0.70 mm to (49.1, 18.9)
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Routing:
- net R/S_OUT(OUT_STAGE_RIGHT): track 48.5 -> 153.5 mm, vias 0 -> 2
- net L/M_OUT(OUT_STAGE_LEFT): track 48.8 -> 151.6 mm, vias 0 -> 2
- net E+_OUT_STAGE_LEFT: track 1.27 -> 73.2 mm, vias 0 -> 1
- net E+_OUT_STAGE_RIGHT: track 1.27 -> 70.9 mm, vias 0 -> 1
- net N$31: track 0.00 -> 62.6 mm, vias 0 -> 2
- net L/M_OUT(VCA1_OUT): track 52.0 -> 110.7 mm, vias 0 -> 3
- net N$28: track 0.00 -> 55.2 mm, vias 0 -> 2
- net N$8: track 0.00 -> 53.6 mm, vias 0 -> 2
- net N$11: track 0.00 -> 53.4 mm, vias 0 -> 2
- net R/S_OUT(VCA2_OUT): track 51.0 -> 101.6 mm, vias 0 -> 4
- net AGND: track 329.5 -> 378.2 mm, vias 96 -> 122
- net N$58: track 64.9 -> 112.4 mm
- net N$59: track 64.4 -> 103.9 mm
- net N$19: track 0.00 -> 37.0 mm
- net R/S_IN(VCA2_IN): track 56.4 -> 91.8 mm, vias 0 -> 2
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
Commit message: BOM CleanUp
Parts:
- R28, R30, R36, R37: value 20k -> 20 k
- R7: value 680R -> 680 R
- R97, R98: value 650 R -> 680 R
- moved R12 0.40 mm to (28.3, 16.1)
- moved LED5 0.30 mm to (81.2, 16.4)
- moved R77 0.14 mm to (186.5, 33.1)
- moved R7 0.10 mm to (52.8, 33.8)
Routing:
- net N$43: track 31.6 -> 29.9 mm
- net -15V_SIG: track 91.0 -> 92.4 mm
- net L/M_OUT(OUT_STAGE_LEFT): track 151.6 -> 152.5 mm
- net OUT6_DRIVER: track 170.2 -> 169.4 mm
- net V-: track 142.0 -> 142.5 mm

Commit message: finished all PCB designs and created output data.
Parts:
- removed ANALOG_VOLT: 90814-0204, electro_mechanical:MOLEX_90814-0204
- added ANALOG_VOLT_IN, ANALOG_VOLT_OUT, DISPLAY2, INSERT_AFTER_GAIN, INSERT_BEFORE_GAIN: 90814-0204, electro_mechanical:MOLEX_90814-0204
- added TP03, TP04, TP05, TP06, TP07, TP08, TP09, TP10: TPTHT, C_Sager_Bibliothek:THT_PIN
- moved R83 8.86 mm to (176.3, 61.7)
- moved R85 8.86 mm to (176.3, 63.8)
- moved R39 8.23 mm to (179.4, 24.4)
- moved R42 5.32 mm to (176.3, 24.4), turned to 0 degrees
- moved R87 1.66 mm to (168.4, 14.8)
- moved R86 1.66 mm to (168.4, 16.9)
- moved R69 0.80 mm to (124.4, 3.50)
- moved R15 0.80 mm to (122.1, 3.50)
- moved C6 0.61 mm to (25.3, 11.4)
- moved C75 0.42 mm to (165.4, 48.8)
- moved LED6 0.10 mm to (6.30, 16.1)
- moved LED7 0.10 mm to (18.9, 16.1)
- renumbered DISPLAY to DISPLAY1
Connections:
- new net L/M_OUT(OUT_STAGE_LEFT)_BEFORE: C38.2, IC11.57, IC5.1, INSERT_AFTER_GAIN.3, R28.2
- new net N$96: INSERT_BEFORE_GAIN.2, R37.1
- new net N$97: INSERT_BEFORE_GAIN.4, R36.1
- new net PB12: IC10.73, TP05.P$1
- new net PD10: IC10.79, TP08.P$1
- new net PD11: IC10.80, TP09.P$1
- new net PD12: IC10.81, TP10.P$1
- new net R/S_OUT(OUT_STAGE_RIGHT)_BEFORE: C37.2, IC11.59, IC5.7, INSERT_AFTER_GAIN.1, R30.2
- new net USART1_RX: DISPLAY2.2, IC10.76
- new net USART1_TX: DISPLAY2.1, IC10.136
- net +5V: now also DISPLAY2.3
- net A_GND_TO_STAR: now also ANALOG_VOLT_IN.3, ANALOG_VOLT_IN.4, ANALOG_VOLT_OUT.3, ANALOG_VOLT_OUT.4; no longer ANALOG_VOLT.3, ANALOG_VOLT.4
- net DIN_DAC: now also TP04.P$1
- net DISPLAY_GND_TO_STAR: now also DISPLAY2.4
- net L/M_OUT(OUT_STAGE_LEFT): now also INSERT_AFTER_GAIN.4; no longer C38.2, IC11.57, IC5.1, R28.2
- net L/M_OUT(VCA1_OUT): now also INSERT_BEFORE_GAIN.3; no longer R36.1
- net R/S_OUT(OUT_STAGE_RIGHT): now also INSERT_AFTER_GAIN.2; no longer C37.2, IC11.59, IC5.7, R30.2
- net R/S_OUT(VCA2_OUT): now also INSERT_BEFORE_GAIN.1; no longer R37.1
- net SCLK_DAC: now also TP03.P$1
- net USART3_RX: now also TP06.P$1
- net USART3_TX: now also TP07.P$1
- net V+: now also ANALOG_VOLT_IN.1, ANALOG_VOLT_OUT.1; no longer ANALOG_VOLT.1
- net V-: now also ANALOG_VOLT_IN.2, ANALOG_VOLT_OUT.2; no longer ANALOG_VOLT.2
Routing:
- net L/M_OUT(OUT_STAGE_LEFT)_BEFORE: track 0.00 -> 134.9 mm, vias 0 -> 4
- net R/S_OUT(OUT_STAGE_RIGHT)_BEFORE: track 0.00 -> 121.3 mm, vias 0 -> 2
- net L/M_OUT(OUT_STAGE_LEFT): track 152.5 -> 50.3 mm, vias 2 -> 3
- net R/S_OUT(OUT_STAGE_RIGHT): track 153.0 -> 51.2 mm
- net USART1_RX: track 0.00 -> 41.0 mm, vias 0 -> 2
- net USART1_TX: track 0.00 -> 35.0 mm, vias 0 -> 2
- net PD12: track 0.00 -> 20.7 mm
- net PD11: track 0.00 -> 18.1 mm
- net SCLK_DAC: track 40.3 -> 58.0 mm
- net A_GND_TO_STAR: track 67.8 -> 84.1 mm
- net PD10: track 0.00 -> 15.2 mm
- net DIN_DAC: track 45.5 -> 60.2 mm
- net DISPLAY_GND_TO_STAR: track 52.5 -> 65.8 mm, vias 0 -> 2
- net USART3_TX: track 0.00 -> 12.1 mm
- net N$96: track 0.00 -> 10.6 mm, vias 0 -> 2
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- added copper zone on layer 16, net LOWER
Other:
- board text added: "Debug1"
- board text added: "Debug2"
- board text added: "PB12"
- board text added: "PD10"
- board text added: "PD11"
- board text added: "PD12"
- board text added: "USART3_RX"
- board text added: "USART3_TX"
