File: electronic/Eagle/quantum/ParmetricEQ/ParametricEQ_V_1_0.sch (EAGLE design)
At the start: 83 parts, among them IC1 OP275_SOIC8, IC14 TL072, IC2 OP275_SOIC8, IC3 OP275_SOIC8, IC4 DAC084S085CIMM_NOPB, IC5 DAC084S085CIMM_NOPB, J1 90814-0204, J2 90814-0204, Q1 TRANSOSTOR_NPN, Q2 TRANSOSTOR_NPN, U1 THAT2181SO8-US, U2 THAT2181SO8-US, U3 THAT2181SO8-US

Commit message: progress on ParametricEQ
Parts:
- added C15, C16, C17: 100 nF, passive components:CAPACITOR_0603
- added C18: 10 uF, passive components:CAPACITOR_1206
- added I2C-CONN, PRG-CONN: 90814-0204, electro_mechanical:90814-0204
- added IC6: STM32F031K6T6, C_Sager_Bibliothek:STM32F031K6T6
- added J10, J3, J4, J5, J6, J7, J8, J9: 10018783-10102TLF, electro_mechanical:10018783-10102TLF
- added R36, R37, R39: 10k, passive components:RESISTOR_0603
- IC14: device C_Sager_Bibliothek:TL072 -> OP-AMPS:TL072
Connections:
- removed net CS_MID1_R: R20.2
- new net +3V3: C15.1, C16.1, C17.1, C18.1, I2C-CONN.3, IC6.VDDA, IC6.VDD_1, IC6.VDD_2
- new net ADRR.1: IC6.PF0-OSC_IN, R39.2
- new net ADRR.2: IC6.PF1-OSC_OUT, R36.2
- new net BOOT_0: IC6.BOOT0, R37.2
- new net I2C1_SCL: I2C-CONN.2, IC6.PB6
- new net I2C1_SDA: I2C-CONN.1, IC6.PA10
- new net NRST: IC6.NRST, PRG-CONN.2
- new net SWCLK: IC6.PA14, PRG-CONN.1
- new net SWDIO: IC6.PA13, PRG-CONN.3
- net CS_MID1_R1: now also R20.2
- net GND: now also C15.2, C16.2, C17.2, C18.2, I2C-CONN.4, IC6.VSS_1, IC6.VSS_2, PRG-CONN.4, R36.1, R37.1, R39.1
Other:
- moved on the sheet: R19, R20, R21
