File: electronic/Eagle/quantum/ParmetricEQ/ParametricMid/ParametricMidPCB_V_1_0.brd (EAGLE design)
At the start: 100 x 140 mm, 101 parts, among them IC1 OP275_SOIC8, IC14 TL072, IC2 OP275_SOIC8, IC3 OP275_SOIC8, IC4 DAC084S085CIMM_NOPB, IC5 DAC084S085CIMM_NOPB, IC6 STM32F031K6T6, J1 90814-0204, J10 10018783-10102TLF, J2 90814-0204, J3 10018783-10102TLF, J4 10018783-10102TLF, J5 10018783-10102TLF, J6 10018783-10102TLF, J7 10018783-10102TLF, J8 10018783-10102TLF, J9 10018783-10102TLF, Q1 TRANSOSTOR_NPN, Q2 TRANSOSTOR_NPN, U1 THAT2181SO8-US, U2 THAT2181SO8-US, U3 THAT2181SO8-US

Commit message: updates ParametricEQ
Parts:
- removed C15, C16, C17, C19: 100 nF, passive components:C0603
- removed C18, C64: 10 uF, passive components:C1206
- removed I2C-CONN, J1, J2, PRG-CONN: 90814-0204, electro_mechanical:MOLEX_90814-0204
- removed IC6: STM32F031K6T6, C_Sager_Bibliothek:QFP80P900X900X160-32N
- removed J10, J3, J4, J5, J6, J7, J8, J9: 10018783-10102TLF, electro_mechanical:1001878310102TLF
- removed R36, R37, R39: 10k, passive components:R0603
- removed R60, R61, R67: 10 k, passive components:R0603
- removed R68: 20 k, passive components:R0603
- removed U$1, U$2: TL072, OP-AMPS:SOIC8
- removed Z1: ZENER_DIODE_BZT, passive components:SODFL1608X65N
Connections:
- removed net +3V3: C15.1, C16.1, C17.1, C18.1, I2C-CONN.3, IC6.1, IC6.17, IC6.5
- removed net 1V_DAC_UNBUFFERD: C19.1, C64.1, R61.2, R68.1, U$2.3
- removed net 2V_DAC_REF: R67.1, R68.2, Z1.1
- removed net ADRR.1: IC6.2, R39.2
- removed net ADRR.2: IC6.3, R36.2
- removed net AGND: C19.2, C64.2, R60.1, Z1.2
- removed net BOOT_0: IC6.31, R37.2
- removed net I2C1_SCL: I2C-CONN.2, IC6.29
- removed net I2C1_SDA: I2C-CONN.1, IC6.20
- removed net L-IN: J2.3
- removed net L-OUT: J2.4
- removed net N$67: R60.2, R61.1, U$2.5
- removed net NRST: IC6.4, PRG-CONN.2
- removed net SWCLK: IC6.24, PRG-CONN.1
- removed net SWDIO: IC6.23, PRG-CONN.3
- net 0,5V_DAC: no longer U$2.6, U$2.7
- net 1V_DAC: no longer U$2.1, U$2.2
- net GND: no longer C15.2, C16.2, C17.2, C18.2, I2C-CONN.4, IC6.16, IC6.32, J1.3, J1.4, PRG-CONN.4, R36.1, R37.1, R39.1
- net MID1_R-IN: no longer J2.1
- net MID1_R-OUT: no longer J2.2
- net V+: no longer J1.1, R67.2, U$1.8, U$2.8
- net V-: no longer J1.2, U$1.4, U$2.4
