File: electronic/Eagle/quantum/ParmetricEQ/BasePCB/BasePCB_V_1_0.brd (EAGLE design)
At the start: 86.3 x 100 mm, 97 parts, among them IC1 OP275_SOIC8, IC14 TL072, IC2 OP275_SOIC8, IC3 OP275_SOIC8, IC4 DAC084S085CIMM_NOPB, IC5 DAC084S085CIMM_NOPB, IC6 STM32F031K6T6, J1 90814-0204, J2 90814-0204, J4 10018783-10102TLF, J5 10018783-10102TLF, J6 10018783-10102TLF, J7 10018783-10102TLF, Q1 TRANSOSTOR_NPN, Q2 TRANSOSTOR_NPN, U1 THAT2181SO8-US, U2 THAT2181SO8-US, U3 THAT2181SO8-US

Commit message: updates ParametricEQ
Parts:
- added J10, J3, J8, J9: 10018784-10210TLF, electro_mechanical:1001878410210TLF
- J4, J5, J6, J7: value 10018783-10102TLF -> 10018784-10210TLF; device electro_mechanical:1001878310102TLF -> electro_mechanical:1001878410210TLF
- moved J4 59.2 mm to (40.0, 80.0)
- moved J6 50.9 mm to (20.0, 80.0)
- moved J5 23.8 mm to (40.0, 10.0)
- moved J7 21.7 mm to (20.0, 10.0)
Other:
- board size 86.3 x 100 mm -> 100 x 140 mm

Commit message: split PCB in ParametricEQ
Parts:
- removed C1, C13, C14, C19, C2, C3, C4, C5, C6, C7, C8: 100 nF, passive components:C0603
- removed C10, C11, C12, C9: (no value), passive components:C0603
- removed C64: 10 uF, passive components:C1206
- removed IC1, IC2, IC3: OP275_SOIC8, OP-AMPS:SOIC8
- removed IC14, U$1, U$2, U$3: TL072, OP-AMPS:SOIC8
- removed IC4, IC5: DAC084S085CIMM_NOPB, SPI:SOP50P490X110-10N
- removed Q1, Q2: TRANSOSTOR_NPN, active components:SOT96P237X111-3N
- removed R1, R2, R3: 5k1, passive components:R0603
- removed R10, R11, R12, R13, R14, R15, R16, R17, R18, R22, R23, R24, R25, R26, R27, R28, R32, R33, R34, R35, R4, R5, R6, R7, R8, R9: (no value), passive components:R0603
- removed R19, R20, R21, R29, R30, R31: 500 R, passive components:R0603
- removed R38, R41, R44: 27 k, passive components:R0603
- removed R40, R43, R63: 160 k, passive components:R0603
- removed R58, R60, R61, R67, R70, R72: 10 k, passive components:R0603
- removed R59: 56 k, passive components:R0603
- removed R68: 20 k, passive components:R0603
- removed S1: ADG436BRZ, analog switches:SOIC127P600X175-16N
- removed U1, U2, U3: THAT2181SO8-US, THAT_Library:SO08
- removed Z1: ZENER_DIODE_BZT, passive components:SODFL1608X65N
- added C20, C22, C24, C26, C28, C30, C32, C34, C37, C39, C41, C43, C45, C47, C49: 10 uF, passive components:C1206
- added C21, C23, C25, C27, C29, C31, C33, C35, C36, C38, C40, C42, C44, C46, C48, C50: 100 nF, passive components:C0603
- added IC10, IC11, IC12, IC13, IC15, IC7, IC8, IC9: DAC084S085CIMM_NOPB, SPI:SOP50P490X110-10N
- added R42, R45, R46, R47, R48, R49, R50, R51, R52, R53, R54, R55, R56, R57, R62, R64, R65, R66, R69, R71, R73, R74, R75, R76: 500 R, passive components:R0603
- C15: value 100 nF -> 10 uF; device passive components:C0603 -> passive components:C1206
- moved C15 149.6 mm to (-64.6, -625.1)
- moved C16 108.4 mm to (-88.9, -591.0)
- moved J5 15.0 mm to (40.0, 25.0), turned to 270 degrees
- moved J7 15.0 mm to (20.0, 25.0), turned to 270 degrees
- moved J8 15.0 mm to (80.0, 25.0), turned to 270 degrees
- moved J9 15.0 mm to (60.0, 25.0), turned to 270 degrees
- moved J10 5.00 mm to (80.0, 75.0)
- moved J3 5.00 mm to (60.0, 75.0)
- moved J4 5.00 mm to (40.0, 75.0)
- moved J6 5.00 mm to (20.0, 75.0)
Connections:
- removed net .: IC14.1, R59.2, R72.2
- removed net 0,5V_DAC: IC14.3, U$2.6, U$2.7
- removed net 1V_DAC: IC4.7, U$2.1, U$2.2
- removed net 1V_DAC_UNBUFFERD: C19.1, C64.1, R61.2, R68.1, U$2.3
- removed net 2V_DAC_REF: R67.1, R68.2, Z1.1
- removed net AGND: C19.2, C64.2, R60.1, Z1.2
- removed net CS_MID1_R1: R20.2, R30.2
- removed net DIN: R19.2
- removed net DIN1: R29.2
- removed net EC+_VCA1_MID1_R: R23.1, U$3.1, U1.2
- removed net EC+_VCA2_MID1_R: R27.1, U$3.7, U2.2
- removed net MID1_R-IN: J2.1, R5.1, S1.2
- removed net MID1_R-OUT: J2.2, S1.3
- removed net MID1_R-PROCESSED: IC1.7, R7.2, S1.4
- removed net MID1_R_BOOST: IC1.6, R6.2, R7.1, S1.10
- removed net MID1_R_BOOST/CUT: Q1.3, R32.1, S1.9
- removed net MID1_R_BYPASS: Q2.3, R34.1, S1.1
- removed net MID1_R_CUT: IC1.2, R4.1, R5.2, S1.12
- removed net MID1_R_GAIN: IC14.6, IC14.7, U3.2
- removed net MID1_R_OUT_C: IC4.4, R70.1
- removed net MID1_R_SIGNAL: R8.1, S1.11
- removed net MID1_R_SYM1: R38.1, R40.2
- removed net MID1_R_SYM2: R41.1, R43.2
- removed net MID1_R_SYM3: R44.1, R63.2
- removed net MID1_R_V_FREQ: IC4.2, R22.2, R28.2
- removed net MID1_R_V_Q: IC4.3, R24.2, R25.2, R26.2
- removed net N$10: C12.2, C9.2, IC2.7, R13.2, R14.1
- removed net N$11: R14.2, U2.1
- removed net N$12: C10.1, IC3.6, U2.8
- removed net N$13: C11.1, IC3.1, R16.1, R8.2
- removed net N$14: C10.2, IC3.7, R15.2
- removed net N$15: C11.2, IC3.2, R16.2, R17.1, U3.8
- removed net N$16: R18.1, U3.1
- removed net N$17: C12.1, R17.2, R18.2
- removed net N$18: IC4.8, R19.1
- removed net N$19: IC4.9, R20.1
- removed net N$20: IC4.10, R21.1
- removed net N$21: R22.1, R23.2, U$3.2
- removed net N$22: R24.1, U$3.3
- removed net N$23: R26.1, R27.2, R28.1, U$3.6
- removed net N$24: IC5.8, R29.1
- removed net N$25: IC5.9, R30.1
- removed net N$26: IC4.5, R33.2
- removed net N$27: IC5.10, R31.1
- removed net N$28: Q2.1, R35.1
- removed net N$29: Q1.1, R33.1
- removed net N$30: IC5.5, R35.2
- removed net N$56: IC5.2, R38.2
- removed net N$57: IC5.3, R41.2
- removed net N$58: IC5.4, R44.2
- removed net N$66: IC14.5, R58.2, R59.1
- removed net N$67: R60.2, R61.1, U$2.5
- removed net N$74: IC14.2, R70.2, R72.1
- removed net N$8: R11.2, U1.1
- removed net N$9: C9.1, IC2.6, U1.8
- removed net SCLK: R21.2
- removed net SCLK1: R31.2
- new net N$31: IC7.8, R42.1
- new net N$32: IC7.9, R45.1
- new net N$33: IC7.10, R46.1
- new net N$34: IC7.2
- new net N$35: IC7.3
- new net N$36: IC7.4
- new net N$37: IC7.5
- new net N$38: IC8.8, R47.1
- new net N$39: IC8.9, R48.1
- new net N$40: IC8.10, R49.1
- new net N$41: IC8.2
- new net N$42: IC8.3
- new net N$43: IC8.4
- new net N$44: IC8.5
- new net N$45: IC9.8, R50.1
- new net N$46: IC9.9, R51.1
- new net N$47: IC9.10, R52.1
- new net N$48: IC9.2
- new net N$49: IC9.3
- new net N$50: IC9.4
- new net N$51: IC9.5
- new net N$52: IC10.8, R53.1
- new net N$53: IC10.9, R54.1
- new net N$54: IC10.10, R55.1
- new net N$55: IC10.2
- new net N$59: IC10.3
- new net N$60: IC10.4
- new net N$61: IC10.5
- new net N$62: IC11.8, R56.1
- new net N$63: IC11.9, R57.1
- new net N$64: IC11.10, R62.1
- new net N$65: IC11.2
- new net N$68: IC11.3
- new net N$69: IC11.4
- new net N$70: IC11.5
- new net N$71: IC12.8, R64.1
- new net N$72: IC12.9, R65.1
- new net N$73: IC12.10, R66.1
- new net N$75: IC12.2
- new net N$76: IC12.3
- new net N$77: IC12.4
- new net N$78: IC12.5
- new net N$79: IC13.8, R69.1
- new net N$80: IC13.9, R71.1
- new net N$81: IC13.10, R73.1
- new net N$82: IC13.2
- new net N$83: IC13.3
- new net N$84: IC13.4
- new net N$85: IC13.5
- new net N$86: IC15.8, R74.1
- new net N$87: IC15.9, R75.1
- new net N$88: IC15.10, R76.1
- new net N$89: IC15.2
- new net N$90: IC15.3
- new net N$91: IC15.4
- new net N$92: IC15.5
- new net R-IN: J2.1
- new net R-OUT: J2.2
- net +3V3: no longer C15.1
- net +5V: now also C15.1, C20.1, C21.1, C22.1, C23.1, C24.1, C25.1, C26.1, C27.1, C28.1, C29.1, C30.1, C31.1, C32.1, C33.1, C34.1, C35.1, C36.1, C37.1, C38.1, C39.1, C40.1, C41.1, C42.1, C43.1, C44.1, C45.1, C46.1, C47.1, C48.1, C49.1, C50.1, IC10.1, IC10.7, IC11.1, IC11.7, IC12.1, IC12.7, IC13.1, IC13.7, IC15.1, IC15.7, IC7.1, IC7.7, IC8.1, IC8.7, IC9.1, IC9.7; no longer IC4.1, IC5.1, IC5.7, R32.2, R34.2
- net GND: now also C20.2, C21.2, C22.2, C23.2, C24.2, C25.2, C26.2, C27.2, C28.2, C29.2, C30.2, C31.2, C32.2, C33.2, C34.2, C35.2, C36.2, C37.2, C38.2, C39.2, C40.2, C41.2, C42.2, C43.2, C44.2, C45.2, C46.2, C47.2, C48.2, C49.2, C50.2, IC10.6, IC11.6, IC12.6, IC13.6, IC15.6, IC7.6, IC8.6, IC9.6; no longer C1.2, C13.2, C14.2, C2.2, C3.2, C4.2, C5.2, C6.2, C7.2, C8.2, IC1.3, IC1.5, IC2.5, IC3.3, IC3.5, IC4.6, IC5.6, Q1.2, Q2.2, R1.1, R10.1, R2.1, R25.1, R3.1, R58.1, S1.6, U$3.5, U1.3, U1.6, U2.3, U2.6, U3.3, U3.6
- net N$1: now also J9.B18; no longer R1.2, U1.5
- net N$2: now also J4.B18; no longer R2.2, U2.5
- net N$3: now also J3.B18; no longer R3.2, U3.5
- net N$4: now also J8.B18; no longer IC2.3, R10.2, R9.2
- net N$5: now also J7.B18; no longer IC1.1, R4.2, R6.1, R9.1
- net N$6: now also J5.B18; no longer IC2.2, R12.1, R13.1, R15.1
- net N$7: now also J6.B18; no longer IC2.1, R11.1, R12.2
- net V+: now also J10.A1, J10.B1, J3.A1, J3.B1, J4.A1, J4.B1, J5.A1, J5.B1, J6.A1, J6.B1, J7.A1, J7.B1, J8.A1, J8.B1, J9.A1, J9.B1; no longer C14.1, C2.1, C3.1, C6.1, C7.1, IC1.8, IC14.8, IC2.8, IC3.8, R67.2, S1.13, U$1.8, U$2.8, U$3.8, U1.7, U2.7, U3.7
- net V-: now also J10.A18, J10.B18, J3.A18, J4.A18, J5.A18, J6.A18, J7.A18, J8.A18, J9.A18; no longer C1.1, C13.1, C4.1, C5.1, C8.1, IC1.4, IC14.4, IC2.4, IC3.4, R40.1, R43.1, R63.1, S1.5, U$1.4, U$2.4, U$3.4
Other:
- board size 100 x 140 mm -> 100 x 100 mm
