File: electronic/Eagle/quantum/EncoderPCB/EncoderPCB_V2_lower/EncoderPCB_V2_lower.sch (EAGLE design)
At the start: 20 parts, among them IC1 STM32F031K6T6

Commit message: progress on parametricEQ
Parts:
- added C5, C6, C7: 100nF, C_Sager_Bibliothek:CAPACITOR"
- added C8: 10 uF, passive components:CAPACITOR_1206
- added IC2: STM32F031K6T6, C_Sager_Bibliothek:STM32F031K6T6
- added PRG-CONN1: 90814-0204, electro_mechanical:90814-0204
- added R5, R6: 10k, passive components:RESISTOR_0603
Connections:
- net +3V3: now also C5.1, C6.1, C7.1, C8.1, IC2.VDDA, IC2.VDD_1, IC2.VDD_2
- net ADRR.: now also IC2.PF1-OSC_OUT, R5.2
- net BOOT_0: now also IC2.BOOT0, R6.2
- net BUTTON_ENC1: now also IC2.PB5
- net BUTTON_ENC2: now also IC2.PB7
- net BUTTON_ENC3: now also IC2.PF0-OSC_IN
- net B_ENC1: now also IC2.PA5
- net B_ENC2: now also IC2.PB0
- net B_ENC3: now also IC2.PB4
- net ENCODER1_A: now also IC2.PA8
- net ENCODER1_B: now also IC2.PA9
- net ENCODER2_A: now also IC2.PA0
- net ENCODER2_B: now also IC2.PA1
- net ENCODER3_A: now also IC2.PA6
- net ENCODER3_B: now also IC2.PA7
- net GND: now also C5.2, C6.2, C7.2, C8.2, IC2.VSS_1, IC2.VSS_2, PRG-CONN1.4, R5.1, R6.1
- net G_ENC1: now also IC2.PA4
- net G_ENC2: now also IC2.PA12
- net G_ENC3: now also IC2.PB3
- net I2C1_SCL: now also IC2.PB6
- net I2C1_SDA: now also IC2.PA10
- net NRST: now also IC2.NRST, PRG-CONN1.2
- net R_ENC1: now also IC2.PA3
- net R_ENC2: now also IC2.PA11
- net R_ENC3: now also IC2.PB1
- net SWCLK: now also IC2.PA14, PRG-CONN1.1
- net SWDIO: now also IC2.PA13, PRG-CONN1.3
- net USART1_RX1: now also IC2.PA15
- net USART1_TX: now also IC2.PA2
Other:
- moved on the sheet: I2C-CONN, PRG-CONN

Commit message: finished EncoderPCB, Implemented Float OSC
Parts:
- removed C2, C7: 100nF, C_Sager_Bibliothek:CAPACITOR"
- removed S5: PEL12T-4225S-S1024, electro_mechanical:PEL12T-4225S-S1024
- added R12, R13, R14, R15, R16, R7: 51 R, passive components:RESISTOR_0603
Connections:
- removed net ADRR.: IC1.PF1-OSC_OUT, IC2.PF1-OSC_OUT, R1.2, R5.2
- removed net BOOT_0: IC1.BOOT0, IC2.BOOT0, R11.2, R6.2
- removed net BUTTON_ENC1: IC1.PB5, IC2.PB5, S1.COM
- removed net BUTTON_ENC2: IC1.PB7, IC2.PB7
- removed net BUTTON_ENC3: IC1.PF0-OSC_IN, IC2.PF0-OSC_IN, S3.COM
- removed net B_ENC1: IC1.PA5, IC2.PA5, R4.1
- removed net B_ENC2: IC1.PB0, IC2.PB0
- removed net B_ENC3: IC1.PB4, IC2.PB4, R10.1
- removed net ENCODER1_A: IC1.PA8, IC2.PA8, S1.A1
- removed net ENCODER1_B: IC1.PA9, IC2.PA9, S1.B1
- removed net ENCODER2_A: IC1.PA0, IC2.PA0
- removed net ENCODER2_B: IC1.PA1, IC2.PA1
- removed net ENCODER3_A: IC1.PA6, IC2.PA6, S3.A1
- removed net ENCODER3_B: IC1.PA7, IC2.PA7, S3.B1
- removed net G_ENC1: IC1.PA4, IC2.PA4, R3.1
- removed net G_ENC2: IC1.PA12, IC2.PA12
- removed net G_ENC3: IC1.PB3, IC2.PB3, R9.1
- removed net NRST: IC1.NRST, IC2.NRST, PRG-CONN.2, PRG-CONN1.2
- removed net R_ENC1: IC1.PA3, IC2.PA3, R2.1
- removed net R_ENC2: IC1.PA11, IC2.PA11
- removed net R_ENC3: IC1.PB1, IC2.PB1, R8.1
- removed net SWCLK: IC1.PA14, IC2.PA14, PRG-CONN.1, PRG-CONN1.1
- removed net SWDIO: IC1.PA13, IC2.PA13, PRG-CONN.3, PRG-CONN1.3
- removed net USART1_RX1: IC1.PA15, IC2.PA15
- removed net USART1_TX: IC1.PA2, IC2.PA2
- new net A_ADRR.: IC1.PF1-OSC_OUT, R1.2
- new net A_BOOT_0: IC1.BOOT0, R11.2
- new net A_BUTTON_ENC1: IC1.PB5, S1.COM
- new net A_BUTTON_ENC2: IC1.PB7, S2.COM
- new net A_BUTTON_ENC3: IC1.PF0-OSC_IN
- new net A_B_ENC1: IC1.PA5, R13.1
- new net A_B_ENC2: IC1.PB0, R10.1
- new net A_B_ENC3: IC1.PB4
- new net A_ENCODER1_A: IC1.PA8, S1.A1
- new net A_ENCODER1_B: IC1.PA9, S1.B1
- new net A_ENCODER2_A: IC1.PA0, S2.A1
- new net A_ENCODER2_B: IC1.PA1, S2.B1
- new net A_ENCODER3_A: IC1.PA6
- new net A_ENCODER3_B: IC1.PA7
- new net A_G_ENC1: IC1.PA4, R12.1
- new net A_G_ENC2: IC1.PA12, R9.1
- new net A_G_ENC3: IC1.PB3
- new net A_NRST: IC1.NRST, PRG-CONN1.2
- new net A_R_ENC1: IC1.PA3, R7.1
- new net A_R_ENC2: IC1.PA11, R8.1
- new net A_R_ENC3: IC1.PB1
- new net A_SWCLK: IC1.PA14, PRG-CONN1.1
- new net A_SWDIO: IC1.PA13, PRG-CONN1.3
- new net A_USART1_RX: IC1.PA15
- new net A_USART1_TX: IC1.PA2
- new net B_ADRR.: IC2.PF1-OSC_OUT, R5.2
- new net B_BOOT_0: IC2.BOOT0, R6.2
- new net B_BUTTON_ENC1: IC2.PB5, S3.COM
- new net B_BUTTON_ENC2: IC2.PB7, S4.COM
- new net B_BUTTON_ENC3: IC2.PF0-OSC_IN
- new net B_B_ENC1: IC2.PA5, R4.1
- new net B_B_ENC2: IC2.PB0, R16.1
- new net B_B_ENC3: IC2.PB4
- new net B_ENCODER1_A: IC2.PA8, S3.A1
- new net B_ENCODER1_B: IC2.PA9, S3.B1
- new net B_ENCODER2_A: IC2.PA0, S4.A1
- new net B_ENCODER2_B: IC2.PA1, S4.B1
- new net B_ENCODER3_A: IC2.PA6
- new net B_ENCODER3_B: IC2.PA7
- new net B_G_ENC1: IC2.PA4, R3.1
- new net B_G_ENC2: IC2.PA12, R15.1
- new net B_G_ENC3: IC2.PB3
- new net B_NRST: IC2.NRST, PRG-CONN.2
- new net B_R_ENC1: IC2.PA3, R2.1
- new net B_R_ENC2: IC2.PA11, R14.1
- new net B_R_ENC3: IC2.PB1
- new net B_SWCLK: IC2.PA14, PRG-CONN.1
- new net B_SWDIO: IC2.PA13, PRG-CONN.3
- new net B_USART1_RX: IC2.PA15
- new net B_USART1_TX: IC2.PA2
- new net N$1: R7.2, S1.-_1
- new net N$2: R12.2, S1.-_2
- new net N$3: R13.2, S1.+_1
- new net N$4: R14.2, S4.-_1
- new net N$5: R15.2, S4.-_2
- new net N$6: R16.2, S4.+_1
- net +3V3: now also R5.1, S2.+_2, S4.+_2; no longer C2.1, C7.1
- net GND: now also S2.C1, S4.C1; no longer C2.2, C7.2, R5.1
- net N$10: now also S3.-_2; no longer S1.-_2
- net N$12: now also S3.+_1; no longer S1.+_1
- net N$15: now also S2.-_1; no longer S3.-_1
- net N$16: now also S2.-_2; no longer S3.-_2
- net N$17: now also S2.+_1; no longer S3.+_1
- net N$9: now also S3.-_1; no longer S1.-_1
Other:
- moved on the sheet: C1, C3, C4, C5, C6, C8, I2C-CONN, IC2, PRG-CONN, PRG-CONN1, R10, R11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
