File: electronic/Eagle/quantum/ParmetricEQ/HighPass/HighPass_V1_0/HighPass_V_1_0.sch (EAGLE design)
At the start: 62 parts, among them IC1 OP275_SOIC8, IC2 OP275_SOIC8, IC3 OP275_SOIC8, IC4 TL072, IC5 TL072, U1 THAT2181SO8-US, U2 THAT2181SO8-US, U3 THAT2181SO8-US

Commit message: finished EncoderPCB, Implemented Float OSC
Parts:
- removed R18, R22, R23, R24, R25, R26, R27, R28: (no value), passive components:RESISTOR_0603
- removed R21: 50 k, electro_mechanical:R_TRIMMER_SMDTC33X2503G
- removed R31: 130 k, passive components:RESISTOR_0603
- removed U3: THAT2181SO8-US, THAT_Library:THAT2181SO8-US
- C10, C11, C12, C9: value (none) -> 100 nF
- R10, R11, R12, R13, R14, R15, R4, R5, R6, R7, R8, R9: value (none) -> 130 k
- R16: value (none) -> 10 k
- R17: value (none) -> 56 k
- R3: value 5k1 -> 130 k
Connections:
- net BUFFERED_DAC4_BYPASS renamed BUFFERED_DAC4
- net DAC1_GAIN renamed DAC1_HIGHPASS_FREQ
- net DAC4_BYPASS renamed DAC4
- removed net AUDIO_PROCESSED: IC1B.OUT, R7.2, S1.S1B
- removed net DAC2_FREQ: PCIE1.B8, R23.1, R24.1
- removed net DAC3_Q: PCIE1.B9, R26.2, R28.1
- removed net DIG_BOOST/CUT: PCIE1.B11, S1.IN2
- removed net E+_VCA3: IC5G$2.-IN, IC5G$2.OUT, U3.EC+
- removed net MID_BOOST: IC1B.-IN, R6.2, R7.1, S1.S2A
- removed net MID_CUT: IC1A.-IN, R4.1, R5.2, S1.S2B
- removed net MID_SIGNAL: R8.1, S1.D2
- removed net N$10: C12.2, C9.2, IC2B.OUT, R13.2, R14.1
- removed net N$12: C10.1, IC3B.-IN, U2.OUT
- removed net N$14: C10.2, IC3B.OUT, R15.2
- removed net N$15: C11.2, IC3A.-IN, R16.2, R17.1, U3.OUT
- removed net N$18: IC4G$1.-IN, R22.1, R23.2
- removed net N$19: IC4G$1.+IN, R25.2, R26.1
- removed net N$21: IC4G$2.-IN, R24.2, R27.1, R28.2
- removed net N$24: R21.2, R31.1
- removed net SYM_VCA3: R31.2, U3.SYM
- new net BUFFERED_DAC3: IC4G$2.-IN, IC4G$2.OUT, S1.IN2
- new net DAC1_HIGHSHELF_GAIN: PCIE1.B8, R17.2
- new net DAC3: IC4G$2.+IN, PCIE1.B9
- new net DIG: PCIE1.B11
- new net HIGH_PASS_IN: R14.1, S1.S1B
- new net HIGH_PASS_OUT: IC2A.OUT, R12.1, R13.2, S1.D2
- new net LOW_SHELF_IN: R11.1, R8.1, S1.S2B
- new net LOW_SHELF_OUT: C11.1, C11.2, IC1B.OUT, R6.2, R7.1, R7.2, R9.2
- net AUDIO_IN: now also S1.D1; no longer R5.1, S1.S1A
- net AUDIO_OUT: now also S1.S1A, S1.S2A; no longer S1.D1
- net E+_VCA1: now also IC4G$1.-IN; no longer R22.2
- net E+_VCA2: now also IC5G$2.-IN, IC5G$2.OUT; no longer IC4G$2.OUT, R27.2
- net GND: now also IC2A.+IN, R16.1; no longer C18.2, IC3A.+IN, IC3B.+IN, IC4G$2.+IN, R10.1, R25.1, U3.EC-, U3.GND
- net N$11: now also C12.1, R10.1, R11.2; no longer R14.2, U2.IN
- net N$13: now also IC2A.-IN, R13.1, R14.2, R15.1; no longer C11.1, IC3A.OUT, R16.1, R8.2
- net N$16: now also C18.2, IC2B.OUT, R15.2; no longer R18.1, U3.IN
- net N$17: now also C18.1, IC2B.-IN, U2.OUT; no longer C12.1, R17.2, R18.2
- net N$3: now also C9.1, IC1A.-IN, R3.1, U1.OUT; no longer R3.2, U3.V-
- net N$4: now also C10.2, IC1B.-IN, R4.2, R6.1, R8.2; no longer IC2A.+IN, R10.2, R9.2
- net N$5: now also C9.2, R3.2, R4.1, R5.1; no longer R4.2, R6.1, R9.1
- net N$6: now also C10.1, R5.2; no longer IC2A.-IN, R12.1, R13.1, R15.1
- net N$7: now also U2.IN; no longer IC2A.OUT, R11.1
- net N$8: now also C12.2, R10.2, R9.1; no longer R11.2
- net N$9: now also IC4G$1.+IN, R16.2, R17.1; no longer C9.1, IC2B.-IN, U1.OUT
- net V+: no longer C18.1, R21.3, U3.V+
- net V-: no longer R21.1, R3.1
Other:
- note added: "High Pass"
- note added: "LowShelf"
- note removed: "Feedback path"
- note removed: "analog signal path"
- moved on the sheet: C10, C11, C12, C17, C18, C19, C9, IC1A, IC1B, IC2A, IC2B, IC4G$1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
