File: electronic/Eagle/quantum/EncoderPCB/EncoderPCB_V1_2/EncoderPCB_V1_2.brd (EAGLE design)
At the start: 37.8 x 61.6 mm, 17 parts, among them IC1 STM32F031K6T6

Commit message: finished Routing EncoderPCB_V1_2
Parts:
- removed I2C-CONN: 90814-0204, electro_mechanical:MOLEX_90814-0204
- added J1: 686104183422, electro_mechanical:686104183422
- moved C3 11.0 mm to (13.7, 37.0), turned to 0 degrees
- moved R1 10.6 mm to (6.20, 21.3), turned to 0 degrees
- moved C2 7.44 mm to (5.10, 37.2)
- moved R11 7.27 mm to (7.90, 23.4)
- moved C1 4.56 mm to (7.30, 26.0), turned to 270 degrees
- moved IC1 4.41 mm to (13.4, 31.0)
- moved C4 3.33 mm to (7.10, 36.6)
- moved PRG-CONN 1.77 mm to (8.10, 17.0)
- moved R2 0.30 mm to (21.7, 46.4)
Connections:
- net +3V3: now also J1.3; no longer I2C-CONN.3
- net GND: now also J1.4; no longer I2C-CONN.4
- net I2C1_SCL: now also J1.2; no longer I2C-CONN.2
- net I2C1_SDA: now also J1.1; no longer I2C-CONN.1
Routing:
- net ENCODER3_A: track 0.00 -> 27.8 mm, vias 0 -> 1
- net R_ENC3: track 0.00 -> 26.1 mm, vias 0 -> 2
- net SWDIO: track 0.00 -> 23.1 mm
- net BUTTON_ENC1: track 0.00 -> 22.7 mm, vias 0 -> 2
- net ENCODER3_B: track 0.00 -> 22.6 mm, vias 0 -> 2
- net ENCODER1_B: track 0.00 -> 19.9 mm
- net NRST: track 0.00 -> 18.2 mm
- net G_ENC1: track 0.00 -> 18.2 mm, vias 0 -> 2
- net R_ENC1: track 0.00 -> 17.8 mm, vias 0 -> 2
- net SWCLK: track 0.00 -> 17.6 mm
- net B_ENC1: track 0.00 -> 15.9 mm
- net GND: track 0.00 -> 15.6 mm, vias 0 -> 7
- net BUTTON_ENC3: track 0.00 -> 15.3 mm, vias 0 -> 1
- net I2C1_SCL: track 0.00 -> 14.2 mm, vias 0 -> 2
- net ENCODER1_A: track 0.00 -> 14.0 mm, vias 0 -> 1
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