File: electronic/Eagle/quantum/EncoderPCB/EncoderPCB_V1_2/EncoderPCB_V1_2.sch (EAGLE design)
At the start: 17 parts, among them IC1 STM32F031K6T6

Commit message: finished Routing EncoderPCB_V1_2
Parts:
- removed I2C-CONN: 90814-0204, electro_mechanical:90814-0204
- added J1: 686104183422, electro_mechanical:686104183422
Connections:
- net +3V3: now also J1.3; no longer I2C-CONN.3
- net GND: now also J1.4; no longer I2C-CONN.4
- net I2C1_SCL: now also J1.2; no longer I2C-CONN.2
- net I2C1_SDA: now also J1.1; no longer I2C-CONN.1
Changed lines of the file:
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@@
 <part name="C2" library="C_Sager_Bibliothek" library_urn="urn:adsk.eagle:library:560098" deviceset="CAPACITOR" device="&quot;" package3d_urn="urn:adsk.eagle:package:576738/3" value="100nF"/>
 <part name="C4" library="passive components" library_urn="urn:adsk.eagle:library:16365137" deviceset="CAPACITOR" device="_1206" package3d_urn="urn:adsk.eagle:package:16431717/2" value="10 uF"/>
-<part name="I2C-CONN" library="electro_mechanical" library_urn="urn:adsk.eagle:library:16388331" deviceset="90814-0204" device="" package3d_urn="urn:adsk.eagle:package:16762552/4"/>
 <part name="GND1" library="supply1" library_urn="urn:adsk.eagle:library:371" deviceset="GND" device=""/>
 <part name="+3V4" library="supply1" library_urn="urn:adsk.eagle:library:371" deviceset="+3V3" device=""/>
 <part name="PRG-CONN" library="electro_mechanical" library_urn="urn:adsk.eagle:library:16388331" deviceset="90814-0204" device="" package3d_urn="urn:adsk.eagle:package:16762552/4"/>
 <part name="GND2" library="supply1" library_urn="urn:adsk.eagle:library:371" deviceset="GND" device=""/>
+<part name="J1" library="electro_mechanical" library_urn="urn:adsk.eagle:library:16388331" deviceset="686104183422" device="" package3d_urn="urn:adsk.eagle:package:18115753/3"/>
 </parts>
 <sheets>
@@
 <attribute name="VALUE" x="110.744" y="79.121" size="1.778" layer="96"/>
 </instance>
-<instance part="I2C-CONN" gate="G$1" x="226.06" y="132.08" smashed="yes">
-<attribute name="NAME" x="229.87" y="139.7" size="1.778" layer="95" align="center-left"/>
-<attribute name="VALUE" x="229.87" y="137.16" size="1.778" layer="96" align="center-left"/>
-</instance>
-<instance part="GND1" gate="1" x="248.92" y="124.46" smashed="yes">
-<attribute name="VALUE" x="246.38" y="121.92" size="1.778" layer="96"/>
-</instance>
-<instance part="+3V4" gate="G$1" x="248.92" y="139.7" smashed="yes">
-<attribute name="VALUE" x="246.38" y="134.62" size="1.778" layer="96" rot="R90"/>
+<instance part="GND1" gate="1" x="228.6" y="142.24" smashed="yes">
+<attribute name="VALUE" x="226.06" y="139.7" size="1.778" layer="96"/>
+</instance>
+<instance part="+3V4" gate="G$1" x="228.6" y="160.02" smashed="yes">
+<attribute name="VALUE" x="226.06" y="154.94" size="1.778" layer="96" rot="R90"/>
 </instance>
 <instance part="PRG-CONN" gate="G$1" x="226.06" y="114.3" smashed="yes">
@@
 <instance part="GND2" gate="1" x="248.92" y="106.68" smashed="yes">
 <attribute name="VALUE" x="246.38" y="104.14" size="1.778" layer="96"/>
+</instance>
+<instance part="J1" gate="G$1" x="187.96" y="154.94" smashed="yes">
+<attribute name="NAME" x="204.47" y="162.56" size="1.778" layer="95" align="center-left"/>
+<attribute name="VALUE" x="204.47" y="160.02" size="1.778" layer="96" align="center-left"/>
 </instance>
 </instances>
@@
 <segment>
 <pinref part="GND1" gate="1" pin="GND"/>
-<wire x1="248.92" y1="127" x2="248.92" y2="129.54" width="0.1524" layer="91"/>
-<pinref part="I2C-CONN" gate="G$1" pin="4"/>
-<wire x1="248.92" y1="129.54" x2="246.38" y2="129.54" width="0.1524" layer="91"/>
+<pinref part="J1" gate="G$1" pin="4"/>
+<wire x1="228.6" y1="144.78" x2="228.6" y2="147.32" width="0.1524" layer="91"/>
+<wire x1="228.6" y1="147.32" x2="208.28" y2="147.32" width="0.1524" layer="91"/>
 </segment>
 <segment>
@@
 <segment>
 <pinref part="+3V4" gate="G$1" pin="+3V3"/>
-<wire x1="248.92" y1="137.16" x2="248.92" y2="132.08" width="0.1524" layer="91"/>
-<pinref part="I2C-CONN" gate="G$1" pin="3"/>
-<wire x1="248.92" y1="132.08" x2="246.38" y2="132.08" width="0.1524" layer="91"/>
+<pinref part="J1" gate="G$1" pin="3"/>
+<wire x1="228.6" y1="157.48" x2="228.6" y2="149.86" width="0.1524" layer="91"/>
+<wire x1="228.6" y1="149.86" x2="208.28" y2="149.86" width="0.1524" layer="91"/>
 </segment>
 </net>
@@
 </segment>
 <segment>
-<pinref part="I2C-CONN" gate="G$1" pin="1"/>
-<wire x1="226.06" y1="132.08" x2="223.52" y2="132.08" width="0.1524" layer="91"/>
-<label x="223.52" y="132.08" size="1.016" layer="95" rot="R180" xref="yes"/>
+<label x="210.82" y="154.94" size="1.016" layer="95" rot="MR180" xref="yes"/>
+<pinref part="J1" gate="G$1" pin="1"/>
+<wire x1="208.28" y1="154.94" x2="210.82" y2="154.94" width="0.1524" layer="91"/>
 </segment>
 </net>
@@
 </segment>
 <segment>
-<pinref part="I2C-CONN" gate="G$1" pin="2"/>
-<wire x1="226.06" y1="129.54" x2="223.52" y2="129.54" width="0.1524" layer="91"/>
-<label x="223.52" y="129.54" size="1.016" layer="95" rot="R180" xref="yes"/>
-</segment>
-</net>
+<label x="210.82" y="152.4" size="1.016" layer="95" rot="MR180" xref="yes"/>
+<pinref part="J1" gate="G$1" pin="2"/>
+<wire x1="210.82" y1="152.4" x2="208.28" y2="152.4" width="0.1524" layer="91"/>
+</segment>
+</net>
